File: temperature-a1/temperature-a1.kicad_sch (KiCad schematic)
At the start: 0 parts

Commit message: Add TMP117, connector, pull-ups and a bypass cap
Parts:
- added C?: 1u, symbol Device:C
- added J?: AFC07-S08ECA-00, symbol Connector_Generic:Conn_01x08
- added R? (x2): ~, symbol Device:R
- added U?: TMP117, symbol tmp117:TMP117
Connections:
- new net GND: C?.2, J?.8 (Pin_8), U?.2 (GND), U?.4 (ADD0)
- new net SCL: J?.2 (Pin_2), R?.2, U?.1 (SCL)
- new net SDA: J?.3 (Pin_3), R?.2, U?.6 (SDA)
- new net VDD: C?.1, J?.1 (Pin_1), R?.1, R?.1, U?.5 (V+)
- new net ~ALERT: J?.7 (Pin_7), U?.3 (ALERT)
- no-connect marks 0 -> 3
Other:
- note added: "I2C Address: TMP116/7 = 0x48 (if ADD0 = GND)"
