File: temperature-a1/temperature-a1.kicad_sch (KiCad schematic)
At the start: 5 parts

Commit message: First revision, drc pass
Parts:
- removed R? (x2): ~, symbol Device:R
- added H2: Breakout Holes, connector:BreakoutHoles, symbol Mechanical:MountingHole
- added T2: Mounting Hole, ruuvitag:MountingHole_3.2mm_M3_Pad_Via, symbol Mechanical:Heatsink_Pad
- C1: renamed from C?; footprint (none) -> ruuvitag:0603_CAP
- J1: renamed from J?; footprint (none) -> connector:RUUVI_CONNECTOR_FFC
- U1: renamed from U?; footprint (none) -> ruuvitag:WSON6
Connections:
- net GND: no longer U1.4 (ADD0)
- net VDD: now also U1.4 (ADD0)
- new net Earth_Clean: T2.1
- new net Earth_Protective: U1.7 (THERMAL)
Other:
- note added: "TMP117 I2C ADD0 PIN CONNECTION 1001000x - Ground 1001001x - V+ 1001010x - SDA 1001011x - SCL M117 I2C address is fixed to 0x44"
- note added: "Temperature Sensor"
- note added: "The thermal pad is not electrically connected to anywhere. ->"
- note removed: "I2C Address: TMP116/7 = 0x48 (if ADD0 = GND)"
- company: (none) -> Ruuvi Innovations Ltd.
- title: (none) -> Temperature Sensor
- moved on the sheet: C1, J1

Commit message: Several minor updates and layout polishing
Parts:
- C1: value 1u -> 1uF 10V 20% X8R 0603
- U1: value TMP117 -> TMP117AIDRVR
Changed lines of the file:
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@@
       (effects (font (size 1.27 1.27)) (justify left))
     )
-    (property "Value" "1u" (id 1) (at 117.475 105.4099 0)
+    (property "Value" "1uF 10V 20% X8R 0603" (id 1) (at 85.725 103.5049 0)
       (effects (font (size 1.27 1.27)) (justify left))
     )
@@
     (in_bom yes) (on_board yes)
     (property "Reference" "U1" (id 0) (at 141.605 93.98 0))
-    (property "Value" "TMP117" (id 1) (at 141.605 96.52 0))
+    (property "Value" "TMP117AIDRVR" (id 1) (at 141.605 96.52 0))
     (property "Footprint" "ruuvitag:WSON6" (id 2) (at 141.605 103.505 0)
       (effects (font (size 1.27 1.27)) hide)
@@
     )
     (path "/8ab0f89b-1159-4064-babc-f4cc7abfb936"
-      (reference "C1") (unit 1) (value "1u") (footprint "ruuvitag:0603_CAP")
+      (reference "C1") (unit 1) (value "1uF 10V 20% X8R 0603") (footprint "ruuvitag:0603_CAP")
     )
     (path "/832defa4-3ee7-4110-ac2e-3ed6464d8359"
@@
     )
     (path "/bbaf25d8-329e-4665-9916-a0b5cb55315a"
-      (reference "U1") (unit 1) (value "TMP117") (footprint "ruuvitag:WSON6")
+      (reference "U1") (unit 1) (value "TMP117AIDRVR") (footprint "ruuvitag:WSON6")
     )
   )
