File: temperature-a1/temperature-a1.kicad_pcb (KiCad board)
At the start: 0 parts

Commit message: First revision, drc pass
Parts:
- added C1: 1u, ruuvitag:0603_CAP, F.Cu at (145.0, 89.6)
- added G***: LOGO, LOGO, B.Cu at (145.0, 99.1)
- added G***: LOGO, LOGO, B.Cu at (145.0, 97.0)
- added H2: Breakout Holes, connector:BreakoutHoles, F.Cu at (145.0, 93.0)
- added J1: AFC07-S08ECA-00, connector:RUUVI_CONNECTOR_FFC, F.Cu at (145.0, 98.0)
- added T2: Mounting Hole, ruuvitag:MountingHole_3.2mm_M3_Pad_Via, F.Cu at (145.0, 81.0)
- added U1: TMP117, ruuvitag:WSON6, F.Cu at (145.0, 87.7)
Routing:
- net /SDA: track 0.00 -> 12.5 mm, vias 0 -> 2
- net VDD: track 0.00 -> 11.5 mm, vias 0 -> 2
- net /SCL: track 0.00 -> 10.0 mm
- net Earth_Clean: track 0.00 -> 9.60 mm
- net /~ALERT: track 0.00 -> 9.18 mm
- net GND: track 0.00 -> 8.66 mm, vias 0 -> 6
- net Earth_Protective: vias 0 -> 3
- added copper zone on B.Cu, net Earth_Clean
- added copper zone on F.Cu, net Earth_Clean
- added copper zone on B.Cu, net Earth_Protective
- added copper zone on B.Cu, net GND
- added copper zone on F.Cu, net GND
Other:
- board outline added: 11 x 25 mm
- copper layers 0 -> 2
