File: temperature-a1/temperature-a1.kicad_pcb (KiCad board)
At the start: 2 copper layers, 11 x 25 mm, 7 parts, among them J1 AFC07-S08ECA-00, T2 Mounting Hole, U1 TMP117

Commit message: Several minor updates and layout polishing
Parts:
- C1: value 1u -> 1uF 10V 20% X8R 0603
- U1: value TMP117 -> TMP117AIDRVR
Routing:
- net VDD: track 11.5 -> 14.2 mm
- net GND: track 8.66 -> 7.27 mm
- net /SDA: track 12.5 -> 11.1 mm
- net Earth_Clean: vias 0 -> 6
Other:
- outline, holes or cut-outs redrawn
